Commit message: replacing zed camera with black and white camera

File: simulator/racecar-simulator/racecar_description/urdf/racecar.xacro (robot description, xacro)
@@ -170,6 +170,6 @@
     <axis xyz="0 0 1" />
   </joint>
-  <!-- zed camera -->
-  <link name="zed_camera_link">
+  <!-- camera -->
+  <link name="camera_link">
     <inertial>
       <mass value="1e-5" />
@@ -180,50 +180,23 @@
       <origin xyz="0 0 0" rpy="0 0 0"/>
       <geometry>
-        <box size="0.033 0.175 0.030"/>
-      </geometry>
-    </collision>
-    <visual>
-      <origin xyz="0 0 0" rpy="0 0 0"/>
-      <geometry>
-        <box size="0.033 0.175 0.030"/>
-      </geometry>
-      <material name="red"/>
-    </visual>
-  </link>
-  <joint name="zed_camera_joint" type="fixed">
+        <box size="0.022 0.04 0.022"/>
+      </geometry>
+    </collision>
+    <visual>
+      <origin xyz="0 0 0" rpy="0 0 0"/>
+      <geometry>
+        <box size="0.022 0.04 0.022"/>
+      </geometry>
+      <material name="white"/>
+    </visual>
+  </link>
+  <joint name="camera_joint" type="fixed">
     <origin xyz="0.390 0 0.04" rpy="0 0 0"/>
     <parent link="chassis"/>
-    <child link="zed_camera_link"/>
+    <child link="camera_link"/>
     <axis xyz="0 0 1" />
     <!-- <limit lower="0.0" upper="0.0" effort="0.0" velocity="0.0" /> -->
   </joint>
-  <!-- zed camera lenses -->
-  <!-- It seems these have to have a non-zero mass to have a camera attached? -->
-  <link name="camera_link"><!-- this needs to match the name in zed_wrapper/zed_tf.launch -->
-    <inertial>
-      <mass value="1e-5" />
-      <origin xyz="0 0 0" rpy="0 0 0"/>
-      <inertia ixx="1e-6" ixy="0" ixz="0" iyy="1e-6" iyz="0" izz="1e-6" />
-    </inertial>
-  </link>
-  <link name="zed_camera_right_link">
-    <inertial>
-      <mass value="1e-5" />
-      <origin xyz="0 0 0" rpy="0 0 0"/>
-      <inertia ixx="1e-6" ixy="0" ixz="0" iyy="1e-6" iyz="0" izz="1e-6" />
-    </inertial>
-  </link>
-  <joint name="zed_camera_left_joint" type="fixed">
-    <origin xyz="0 0.06 0" rpy="0 0 0"/>
-    <parent link="zed_camera_link"/>
-    <child link="camera_link"/>
-    <axis xyz="0 0 1" />
-  </joint>
-  <joint name="zed_camera_right_joint" type="fixed">
-    <origin xyz="0 -0.06 0" rpy="0 0 0"/>
-    <parent link="zed_camera_link"/>
-    <child link="zed_camera_right_link"/>
-    <axis xyz="0 0 1" />
-  </joint>
+  <xacro:property name="camera_link"/>
   <!-- Add the remaining xacros -->
   <xacro:include filename="$(find racecar_description)/urdf/racecar.gazebo" />

Commit message: Editing racecar default initial pose & lidar joint position.

File: simulator/racecar-simulator/racecar_description/urdf/racecar.xacro (robot description, xacro)
@@ -165,5 +165,5 @@
   </link>
   <joint name="hokuyo_joint" type="fixed">
-    <origin xyz="0.265 0.0 0.075" rpy="0 0 0"/>
+    <origin xyz="0.265 0.0 0.115" rpy="0 0 0"/>
     <parent link="chassis" />
     <child link="laser" />

Commit message: Updating packages to work conveniently with changed namespaces + More-than-one vehicle navigation + Inter-vehicle Communication

File: simulator/racecar-simulator/racecar_description/urdf/racecar.xacro (robot description, xacro)
@@ -34,5 +34,5 @@
       <material name="black" />
     </visual>
-    <collision>robot
+    <collision>
       <xacro:left_wheels_collision_geometry />
     </collision>
@@ -192,5 +192,5 @@
   </link>
   <joint name="camera_joint" type="fixed">
-    <origin xyz="0.390 0 0.04" rpy="0 0 0"/>
+    <origin xyz="0.390 0 0.08" rpy="0 -0.4 0"/>
     <parent link="chassis"/>
     <child link="camera_link"/>
