Commit message: Updating the vehicle descriptions (modifying the laser link).

File: simulator/racecar-simulator/racecar_description/urdf/ambulance.xacro (robot description, xacro)
@@ -150,10 +150,4 @@
       <xacro:hokuyo_inertial_params />
     </inertial>
-    <collision>
-      <origin xyz="0 0 0" rpy="0 0 0"/>
-      <geometry>
-        <box size="0.1 0.1 0.1"/>
-      </geometry>
-    </collision>
     <visual>
       <origin xyz="0 0 0" rpy="0 0 0"/>

File: simulator/racecar-simulator/racecar_description/urdf/racecar.xacro (robot description, xacro)
@@ -150,10 +150,4 @@
       <xacro:hokuyo_inertial_params />
     </inertial>
-    <collision>
-      <origin xyz="0 0 0" rpy="0 0 0"/>
-      <geometry>
-        <box size="0.1 0.1 0.1"/>
-      </geometry>
-    </collision>
     <visual>
       <origin xyz="0 0 0" rpy="0 0 0"/>
